File: hardware/NRF52 CTAP Authenticator.brd (EAGLE design)
At the start: 60 x 45 mm, 58 parts, among them IC1 LSM6DS33, IC2 GD25Q16, J1 U.FL-R-SMT(10), Q1_1 DMG2305, Q2_1 MMBT2222A, Q5_1 BSS138, U1 APDS-9960, U2 AP2112(3.3V), U3 MCP73831T-2ACI/OT, X2 CON_JST_PH_2PIN_MTPH2

Commit message: hardware revison 2
Connections:
- removed net AREF: J2.2, MDBT50Q-1MV2.12
- net 3.3V: now also J2.2
Routing:
- net AREF: track 22.0 -> 0.00 mm, vias 3 -> 0
- net 3.3V: track 177.6 -> 192.5 mm, vias 2 -> 3
- net GND: track 31.0 -> 33.7 mm
- net SWITCH_A: track 15.0 -> 15.8 mm
- net RESET: track 32.7 -> 33.3 mm
Changed lines of the file:
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@@
 <via x="3.5" y="10.5" extent="1-16" drill="0.3937"/>
 <via x="14.5" y="5" extent="1-16" drill="0.3937"/>
-<via x="17" y="9.5" extent="1-16" drill="0.3937"/>
+<via x="17.73" y="9.67" extent="1-16" drill="0.3937"/>
 <via x="17" y="12" extent="1-16" drill="0.3937"/>
 <via x="13.559" y="15.615" extent="1-16" drill="0.3937"/>
@@
 <via x="57.6" y="6.66" extent="1-16" drill="0.3937"/>
 <via x="37.74" y="3.28" extent="1-16" drill="0.3937"/>
-<via x="21.43" y="4.3" extent="1-16" drill="0.3937"/>
 <wire x1="3.75" y1="15.85" x2="4.85" y2="15.85" width="0.2032" layer="1"/>
 <via x="7" y="6.5" extent="1-16" drill="0.3937"/>
 <via x="19.5" y="13" extent="1-16" drill="0.3937"/>
 <via x="19.5" y="15.5" extent="1-16" drill="0.3937"/>
-<wire x1="6.07" y1="22.59" x2="4.191" y2="21.717" width="0" layer="19" extent="1-1"/>
+<via x="10" y="12.5" extent="1-16" drill="0.3937"/>
+<wire x1="6.07" y1="22.59" x2="5.78865" y2="22.30865" width="0.2032" layer="16"/>
+<wire x1="5.78865" y1="22.30865" x2="5.78865" y2="21.92344375" width="0.2032" layer="16"/>
+<wire x1="5.78865" y1="21.92344375" x2="5.37470625" y2="21.5095" width="0.2032" layer="16"/>
+<wire x1="5.37470625" y1="21.5095" x2="4.78929375" y2="21.5095" width="0.2032" layer="16"/>
+<wire x1="4.78929375" y1="21.5095" x2="4.58179375" y2="21.717" width="0.2032" layer="16"/>
+<wire x1="4.58179375" y1="21.717" x2="4.191" y2="21.717" width="0.2032" layer="16"/>
 </signal>
 <signal name="VBUS" class="1">
@@
 <wire x1="34.59495" y1="23.5" x2="40.15385" y2="29.0589" width="0.4064" layer="1"/>
 <wire x1="40.15385" y1="29.0589" x2="40.15385" y2="29.58655" width="0.4064" layer="1"/>
+<contactref element="J2" pad="2"/>
+<via x="17.5" y="7" extent="1-16" drill="0.3937"/>
+<wire x1="22.32470625" y1="12.142" x2="21.85125" y2="11.66854375" width="0.4064" layer="1"/>
+<wire x1="24" y1="12.45" x2="23.692" y2="12.142" width="0.4064" layer="1"/>
+<wire x1="23.692" y1="12.142" x2="22.32470625" y2="12.142" width="0.4064" layer="1"/>
+<wire x1="21.85125" y1="11.66854375" x2="21.85125" y2="11.35125" width="0.4064" layer="1"/>
+<wire x1="21.85125" y1="11.35125" x2="17.5" y2="7" width="0.4064" layer="1"/>
+<wire x1="17.5" y1="7" x2="19.631" y2="4.869" width="0.4064" layer="16"/>
+<wire x1="19.631" y1="4.869" x2="19.631" y2="1.945" width="0.4064" layer="16"/>
 <wire x1="32.502" y1="15.44" x2="32.502" y2="15.94" width="0" layer="19" extent="1-1"/>
 <wire x1="32.502" y1="13.44" x2="32.502" y2="14.94" width="0" layer="19" extent="1-1"/>
@@
 <wire x1="10.91935" y1="20.1467" x2="10.91935" y2="24.18585" width="0.2032" layer="1"/>
 <wire x1="12.6732" y1="18.39285" x2="10.91935" y2="20.1467" width="0.2032" layer="1"/>
-<wire x1="12.6542" y1="12.0419" x2="12.6542" y2="12.4501" width="0.2032" layer="16"/>
 <wire x1="12.6542" y1="12.4501" x2="12.6732" y2="12.4691" width="0.2032" layer="16"/>
 <wire x1="12.6732" y1="18.39285" x2="12.6732" y2="12.4691" width="0.2032" layer="16"/>
-<wire x1="22.14485" y1="2.55125" x2="12.6542" y2="12.0419" width="0.2032" layer="16"/>
-<wire x1="22.14485" y1="1.945840625" x2="22.14485" y2="2.55125" width="0.2032" layer="16"/>
+<wire x1="22.14485" y1="4.05125" x2="13.746" y2="12.4501" width="0.2032" layer="16"/>
+<wire x1="12.6542" y1="12.4501" x2="13.746" y2="12.4501" width="0.2032" layer="16"/>
+<wire x1="22.14485" y1="1.945840625" x2="22.14485" y2="4.05125" width="0.2032" layer="16"/>
 <wire x1="10.91935" y1="24.18585" x2="10.85" y2="24.25" width="0.2032" layer="1"/>
 <wire x1="22.14485" y1="1.945840625" x2="22.171" y2="1.945" width="0.2032" layer="16"/>
@@
 <contactref element="MDBT50Q-1MV2" pad="4"/>
 <wire x1="7.3476" y1="14.6952" x2="7.3476" y2="15.81775" width="0.2032" layer="1"/>
-<wire x1="7.3476" y1="14.46085" x2="7.3476" y2="14.6952" width="0.2032" layer="16"/>
-<wire x1="11.763" y1="9.979" x2="11.763" y2="10.04545" width="0.2032" layer="16"/>
-<wire x1="11.763" y1="10.04545" x2="7.3476" y2="14.46085" width="0.2032" layer="16"/>
+<wire x1="7.3476" y1="12.96085" x2="7.3476" y2="14.6952" width="0.2032" layer="16"/>
+<wire x1="11.763" y1="9.979" x2="10.32945" y2="9.979" width="0.2032" layer="16"/>
+<wire x1="10.32945" y1="9.979" x2="7.3476" y2="12.96085" width="0.2032" layer="16"/>
 <wire x1="7.3476" y1="15.81775" x2="7.25" y2="15.85" width="0.2032" layer="1"/>
 <wire x1="11.53165" y1="9.7968" x2="11.53165" y2="3.16355" width="0.2032" layer="16"/>
@@
 <via x="37.7585" y="38.1667" extent="1-16" drill="0.3937"/>
 </signal>
-<signal name="AREF">
-<contactref element="MDBT50Q-1MV2" pad="12"/>
-<contactref element="J2" pad="2"/>
-<via x="11.8024" y="15.04673125" extent="1-16" drill="0.3937"/>
-<wire x1="10.84966875" y1="15.04673125" x2="10.4434" y2="15.453" width="0.2032" layer="1"/>
-<wire x1="10.84966875" y1="15.04673125" x2="11.8024" y2="15.04673125" width="0.2032" layer="1"/>
-<wire x1="11.8024" y1="15.04673125" x2="11.8024" y2="13.32456875" width="0.2032" layer="16"/>
-<wire x1="11.8024" y1="13.32456875" x2="11.95481875" y2="13.17215" width="0.2032" layer="16"/>
-<via x="11.95481875" y="13.17215" extent="1-16" drill="0.3937"/>
-<wire x1="11.95481875" y1="13.17215" x2="9.87" y2="11.08733125" width="0.2032" layer="1"/>
-<wire x1="9.87" y1="11.08733125" x2="9.87" y2="10.32" width="0.2032" layer="1"/>
-<wire x1="9.87" y1="10.32" x2="13.1178" y2="7.0722" width="0.2032" layer="1"/>
-<wire x1="15.45304375" y1="7.0722" x2="15.75149375" y2="7.37065" width="0.2032" layer="1"/>
-<via x="15.75149375" y="7.37065" extent="1-16" drill="0.3937"/>
-<wire x1="15.75149375" y1="7.37065" x2="19.631" y2="3.49114375" width="0.2032" layer="16"/>
-<wire x1="19.631" y1="3.49114375" x2="19.631" y2="1.945" width="0.2032" layer="16"/>
-<wire x1="13.1178" y1="7.0722" x2="15.45304375" y2="7.0722" width="0.2032" layer="1"/>
-<wire x1="10.4434" y1="15.453" x2="10.4434" y2="15.8434" width="0.2032" layer="1"/>
-<wire x1="10.4434" y1="15.8434" x2="10.45" y2="15.85" width="0.2032" layer="1"/>
-</signal>
 </signals>
