File: hardware/NRF52 CTAP Authenticator.sch (EAGLE design)
At the start: 58 parts, among them IC1 LSM6DS33, IC2 GD25Q16, J1 U.FL-R-SMT(10), Q1_1 DMG2305, Q2_1 MMBT2222A, Q5_1 BSS138, U1 APDS-9960, U2 AP2112(3.3V), U3 MCP73831T-2ACI/OT, X2 CON_JST_PH_2PIN_MTPH2

Commit message: hardware revison 2
Connections:
- removed net AREF: J2.2, MDBT50Q-1MV2.P0.31/AIN7
- net 3.3V: now also J2.2
